Commit message: plotting works

File: IK/BITL.urdf (robot description, URDF)
Before this commit: robot Patrick, 6 links, 5 joints
Links:
- removed link Base
- added link base_link; visual cylinder length=0.035 radius=0.20
Joints:
- joint BaseJoint: parent Base -> base_link

Commit message: fixed plotting => removing widgets

File: IK/BITL.urdf (robot description, URDF)
Before this commit: robot Patrick, 6 links, 5 joints
Joints:
- joint BaseJoint: limit (none) -> lower=-1.57 upper=1.57

Commit message: tuned joint limits

File: IK/BITL.urdf (robot description, URDF)
Before this commit: robot Patrick, 6 links, 5 joints
Joints:
- joint BaseJoint: limit lower=-1.57 upper=1.57 -> lower=-2.356 upper=2.356
- joint Lower_joint: limit lower=-1.57 upper=1.57 -> lower=0 upper=1.57
- joint Upper_joint: limit lower=-1.57 upper=1.57 -> lower=0 upper=1.57

Commit message: t werkt nimeer

File: IK/BITL.urdf (robot description, URDF)
Before this commit: robot Patrick, 6 links, 5 joints
Links:
- removed link Gripper
- removed link Gripper_rotation
- link Arm_base: geometry visual cylinder length=0.087 radius=0.06
- link Lower_arm: geometry visual cylinder length=0.155 radius=0.03
- link Upper_arm: geometry visual cylinder length=0.12 radius=0.03
- link base_link: geometry visual cylinder length=0.01 radius=0.20
Joints:
- removed joint Arm_joint
- removed joint Arm_rotation
- joint BaseJoint: origin xyz=0.0 0.0 0.067 rpy=0.0 0.0 0.0 -> xyz=0.0 0.0 0.05 rpy=0.0 0.0 0.0
- joint Lower_joint: origin xyz=0.0 0.0 0.05 -> xyz=0.0 0.0 0.044

Commit message: bit of a late commit, but it works

File: IK/BITL.urdf (robot description, URDF)
Before this commit: robot Patrick, 4 links, 3 joints
Joints:
- removed joint BaseJoint
- added joint Base_to_Arm: type revolute, parent base_link, child Arm_base, origin xyz=0.0 0.0 0.05 rpy=0.0 0.0 0.0, axis 0.0 0.0 1, limit lower=-3.14 upper=3.14 effort=100 velocity=1
